File: computer.kicad_pcb (KiCad board)
At the start: 2 copper layers, 102.9 x 58.4 mm, 17 parts

Commit message: Tidying
Parts:
- JP1: renamed from XTAL EN
- R1, R2, R3: value 1k -> 10k
- X1: renamed from 1MHZ XTAL
- renumbered EXP1 to J1, EXP2 to J2, RESET to SW1, CPU to U1, ROM to U2, RAM to U3, XOR to U4, DS1813 to U5
Changed lines of the file:
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@@
     (descr https://www.omron.com/ecb/products/pdf/en-b3f.pdf)
     (tags "tact sw push 6mm")
-    (fp_text reference RESET (at 3.175 6.985) (layer F.SilkS)
+    (fp_text reference SW1 (at 3.175 6.985) (layer F.SilkS)
       (effects (font (size 1 1) (thickness 0.15)))
     )
@@
     (descr "Through hole angled pin header, 1x02, 2.54mm pitch, 6mm pin length, single row")
     (tags "Through hole angled pin header THT 1x02 2.54mm single row")
-    (fp_text reference "XTAL EN" (at 11.43 1.27 180) (layer F.SilkS)
+    (fp_text reference JP1 (at 11.43 1.27 180) (layer F.SilkS)
       (effects (font (size 1 1) (thickness 0.15)))
     )
@@
     (descr "28-lead though-hole mounted DIP package, row spacing 15.24 mm (600 mils), Socket")
     (tags "THT DIP DIL PDIP 2.54mm 15.24mm 600mil Socket")
-    (fp_text reference ROM (at 7.62 35.56) (layer F.SilkS)
+    (fp_text reference U2 (at 7.62 35.56) (layer F.SilkS)
       (effects (font (size 1 1) (thickness 0.15)))
     )
@@
     (descr "TO-92 horizontal, leads in-line, narrow, oval pads, drill 0.75mm (see NXP sot054_po.pdf)")
     (tags "to-92 sc-43 sc-43a sot54 PA33 transistor")
-    (fp_text reference DS1813 (at 1.27 10.16) (layer F.SilkS)
+    (fp_text reference U5 (at 1.27 10.16) (layer F.SilkS)
       (effects (font (size 1 1) (thickness 0.15)))
     )
@@
       (effects (font (size 1 1) (thickness 0.15)))
     )
-    (fp_text value 1k (at 5.08 2.37) (layer F.Fab)
+    (fp_text value 10k (at 5.08 2.37) (layer F.Fab)
       (effects (font (size 1 1) (thickness 0.15)))
     )
@@
       (effects (font (size 1 1) (thickness 0.15)))
     )
-    (fp_text value 1k (at 5.08 2.37) (layer F.Fab)
+    (fp_text value 10k (at 5.08 2.37) (layer F.Fab)
       (effects (font (size 1 1) (thickness 0.15)))
     )
@@
       (effects (font (size 1 1) (thickness 0.15)))
     )
-    (fp_text value 1k (at 5.08 2.37) (layer F.Fab)
+    (fp_text value 10k (at 5.08 2.37) (layer F.Fab)
       (effects (font (size 1 1) (thickness 0.15)))
     )
@@
     (descr "Oscillator, DIP8,http://cdn-reichelt.de/documents/datenblatt/B400/OSZI.pdf")
     (tags oscillator)
-    (fp_text reference "1MHZ XTAL" (at 3.81 -11.26) (layer F.SilkS)
+    (fp_text reference X1 (at 3.81 -11.26) (layer F.SilkS)
       (effects (font (size 1 1) (thickness 0.15)))
     )
@@
     (descr "Through hole straight pin header, 2x20, 2.54mm pitch, double rows")
     (tags "Through hole pin header THT 2x20 2.54mm double row")
-    (fp_text reference EXP2 (at 1.27 50.8) (layer F.SilkS)
+    (fp_text reference J2 (at 1.27 50.8) (layer F.SilkS)
       (effects (font (size 1 1) (thickness 0.15)))
     )
@@
     (descr "14-lead though-hole mounted DIP package, row spacing 7.62 mm (300 mils), Socket")
     (tags "THT DIP DIL PDIP 2.54mm 7.62mm 300mil Socket")
-    (fp_text reference XOR (at 3.81 17.78) (layer F.SilkS)
+    (fp_text reference U4 (at 3.81 17.78) (layer F.SilkS)
       (effects (font (size 1 1) (thickness 0.15)))
     )
@@
     (descr "28-lead though-hole mounted DIP package, row spacing 15.24 mm (600 mils), Socket")
     (tags "THT DIP DIL PDIP 2.54mm 15.24mm 600mil Socket")
-    (fp_text reference RAM (at 8.255 35.56) (layer F.SilkS)
+    (fp_text reference U3 (at 8.255 35.56) (layer F.SilkS)
       (effects (font (size 1 1) (thickness 0.15)))
     )
@@
     (descr "40-lead though-hole mounted DIP package, row spacing 15.24 mm (600 mils), Socket")
     (tags "THT DIP DIL PDIP 2.54mm 15.24mm 600mil Socket")
-    (fp_text reference CPU (at 7.62 50.8) (layer F.SilkS)
+    (fp_text reference U1 (at 7.62 50.8) (layer F.SilkS)
       (effects (font (size 1 1) (thickness 0.15)))
     )
@@
     (descr "Through hole straight pin header, 2x20, 2.54mm pitch, double rows")
     (tags "Through hole pin header THT 2x20 2.54mm double row")
-    (fp_text reference EXP1 (at 1.27 50.8) (layer F.SilkS)
-      (effects (font (size 1 1) (thickness 0.15)))
-    )
+    (fp_text reference J1 (at 1.27 50.8) (layer F.SilkS)
+      (effects (font (size 1 1) (thickness 0.15)))
+    )

Commit message: More tidying up
Parts:
- C1, C2, C3, C4: footprint Capacitor_THT:C_Rect_L7.2mm_W2.5mm_P5.00mm_FKS2_FKP2_MKS2_MKP2 -> Capacitor_THT:C_Disc_D6.0mm_W2.5mm_P5.00mm
- moved C3 5.08 mm to (137.2, 30.5)
- moved C1 5.08 mm to (91.4, 30.5)
- moved C2 5.08 mm to (114.3, 30.5)
- moved C4 1.27 mm to (156.2, 30.5)
Routing:
- net +5V: track 85.5 -> 101.6 mm, vias 10 -> 8
Other:
- board size 102.9 x 58.4 mm -> 104.1 x 67.3 mm
- board text added: "6502 Modular PC - Main board"
