File: main-board/main-board.sch (KiCad schematic (older format))
At the start: 18 parts, among them J1 EXP, J2 EXP, SW1 RESET, U1 W65C02S, U2 28C256, U3 AS6C62256, U4 74HC30, U5 74HC00, U6 DS1813, X1 1MHz

Commit message: remove old peripheral boards, begn new vga design
Parts:
- removed U2: 28C256, Package_DIP:DIP-28_W15.24mm_Socket, symbol Memory_EEPROM:28C256
- removed U4: 74HC30, Package_DIP:DIP-14_W7.62mm_Socket, symbol 74xx:74LS30
- removed unit 2 of U5
- added U2: SST39SF010, Package_DIP:DIP-32_W15.24mm_Socket, symbol Memory_Flash:SST39SF010
- renumbered U5 to U4
Connections:
- net !P_SELECT is gone; now on net GND: J1.12 (Pin_12), J2.12 (Pin_12)
- net !IRQ: now also J1.3 (Pin_3), J2.3 (Pin_3); no longer J1.5 (Pin_5), J2.5 (Pin_5)
- net !NMI: now also J1.4 (Pin_4), J2.4 (Pin_4); no longer J1.6 (Pin_6), J2.6 (Pin_6)
- net !RAM_SELECT: now also J1.28 (Pin_28), J2.28 (Pin_28), U1.25 (A15), U4.2
- net !READ: now also J1.5 (Pin_5), J2.5 (Pin_5), U2.24 (OE); no longer J1.7 (Pin_7), J2.7 (Pin_7)
- net !RESET: now also J1.8 (Pin_8), J2.8 (Pin_8); no longer J1.10 (Pin_10), J2.10 (Pin_10)
- net !ROM_SELECT: now also U2.22 (CE)
- net !WRITE: now also J1.6 (Pin_6), J2.6 (Pin_6); no longer J1.8 (Pin_8), J2.8 (Pin_8)
- net +5V: now also U2.31 (PGM), U2.32 (VCC)
- net A0: now also U2.12 (A0)
- net A1: now also U2.11 (A1)
- net A10: now also U2.23 (A10)
- net A11: now also U2.25 (A11)
- net A12: now also U2.4 (A12)
- net A13: now also U2.28 (A13)
- net A14: now also U4.1
- net A2: now also U2.10 (A2)
- net A3: now also U2.9 (A3)
- net A4: now also U2.8 (A4)
- net A5: now also U2.7 (A5)
- net A6: now also U2.6 (A6)
- net A7: now also U2.5 (A7)
- net A8: now also U2.27 (A8)
- net A9: now also U2.26 (A9)
- net CLK: now also J1.10 (Pin_10), J2.10 (Pin_10); no longer J1.2 (Pin_2), J2.2 (Pin_2)
- net D0: now also U2.13 (D0)
- net D1: now also U2.14 (D1)
- net D2: now also U2.15 (D2)
- net D3: now also U2.17 (D3)
- net D4: now also U2.18 (D4)
- net D5: now also U2.19 (D5)
- net D6: now also U2.20 (D6)
- net D7: now also U2.21 (D7)
- net GND: now also J1.11 (Pin_11), J2.11 (Pin_11), U2.16 (GND), U2.2 (A16), U2.29 (A14), U2.3 (A15); no longer J1.1 (Pin_1), J2.1 (Pin_1)
- net PHI1: now also J1.1 (Pin_1), J2.1 (Pin_1); no longer J1.3 (Pin_3), J2.3 (Pin_3)
- net PHI2: now also J1.2 (Pin_2), J2.2 (Pin_2); no longer J1.4 (Pin_4), J2.4 (Pin_4)
- net R!W: now also J1.7 (Pin_7), J2.7 (Pin_7); no longer J1.9 (Pin_9), J2.9 (Pin_9)
- net RDY: now also J1.9 (Pin_9), J2.9 (Pin_9); no longer J1.11 (Pin_11), J2.11 (Pin_11)
- removed net A15: J1.28 (Pin_28), J2.28 (Pin_28), U1.25 (A15), U4.1, U4.2
- no-connect marks 4 -> 6
Other:
- moved on the sheet: J1, J2, U4A, U4C, U4D
