File: vga-board/vga-board.sch (KiCad schematic (older format))
At the start: 31 parts, among them U1 74HC244, U10 74HC163, U11 74LS158, U12 74LS251, U13 74HC244, U14 74HC244, U15 74HC244, U16 GAL22V10, U17 GAL22V10, U18 GAL22V10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

Commit message: Integtrate IO into mail board, begion VGA layout
Parts:
- added J1, J2: Conn_02x20_Odd_Even, Connector_PinSocket_2.54mm:PinSocket_2x20_P2.54mm_Vertical, symbol Connector_Generic:Conn_02x20_Odd_Even
- J3: renamed from J?; footprint (none) -> Connector_Dsub:DSUB-15-HD_Female_Horizontal_P2.29x1.98mm_EdgePinOffset3.03mm_Housed_MountingHolesOffset4.94mm
- R1, R2, R3, R4, R5, R6: footprint (none) -> Resistor_THT:R_Axial_DIN0207_L6.3mm_D2.5mm_P10.16mm_Horizontal
Connections:
- net HBLANK_END is gone; now on net LINE_INC: U17.20 (IO4)
- net HBLANK_START is gone; now on net !HRST: U17.21 (I03)
- net HSYNC_END is gone; now on net HBLANK: U17.22 (IO2)
- net HSYNC_START is gone; now on net HSYNC: U17.23 (IO1)
- net VBLANK_END is gone; now on net !VRST: U18.20 (IO4)
- net VBLANK_START is gone; now on net BLANK: U18.21 (I03)
- net VSYNC_END is gone; now on net VSYNC: U18.22 (IO2)
- net VSYNC_START is gone; now on net HBLANK: U18.23 (IO1)
- net !HRST: no longer U17.17 (IO7)
- net !VRST: no longer U18.17 (IO7)
- net +5V: now also J1.3 (Pin_3), J1.4 (Pin_4)
- net A0: now also J1.17 (Pin_17)
- net A1: now also J1.18 (Pin_18)
- net A10: now also J1.27 (Pin_27)
- net A11: now also J1.28 (Pin_28)
- net A12: now also J1.29 (Pin_29)
- net A13: now also J1.30 (Pin_30)
- net A14: now also J1.31 (Pin_31)
- net A15: now also J1.32 (Pin_32)
- net A2: now also J1.19 (Pin_19)
- net A3: now also J1.20 (Pin_20)
- net A4: now also J1.21 (Pin_21)
- net A5: now also J1.22 (Pin_22)
- net A6: now also J1.23 (Pin_23)
- net A7: now also J1.24 (Pin_24)
- net A8: now also J1.25 (Pin_25)
- net A9: now also J1.26 (Pin_26)
- net BLANK: no longer U18.16 (IO8)
- net CLK: now also U17.4 (I4), J1.6 (Pin_6); no longer U17.3 (I3)
- net D0: now also J1.33 (Pin_33)
- net D1: now also J1.34 (Pin_34)
- net D2: now also J1.35 (Pin_35)
- net D3: now also J1.36 (Pin_36)
- net D4: now also J1.37 (Pin_37)
- net D5: now also J1.38 (Pin_38)
- net GND: now also J1.1 (Pin_1), J1.2 (Pin_2)
- net HBLANK: no longer U17.18 (IO6), U18.13 (I12)
- net HSYNC: no longer U17.19 (IO5)
- net LINE_INC: no longer U17.16 (IO8)
- net R!W: now also J1.11 (Pin_11)
- net VCLK: now also U17.1 (I1/CLK), U18.1 (I1/CLK)
- net VSYNC: no longer U18.19 (IO5)
- net X0: now also U17.2 (I2); no longer U17.1 (I1/CLK)
- net X1: now also U17.3 (I3); no longer U17.2 (I2)
- net X10: now also U17.13 (I12); no longer U17.11 (I11)
- net X3: now also U17.5 (I5); no longer U17.4 (I4)
- net X4: now also U17.6 (I6); no longer U17.5 (I5)
- net X5: now also U17.7 (I7); no longer U17.6 (I6)
- net X6: now also U17.8 (I8); no longer U17.7 (I7)
- net X7: now also U17.9 (I9); no longer U17.8 (I8)
- net X8: now also U17.10 (I10); no longer U17.9 (I9)
- net X9: now also U17.11 (I11); no longer U17.10 (I10)
- net Y0: now also U18.2 (I2); no longer U18.1 (I1/CLK)
- net Y1: now also U18.3 (I3); no longer U18.2 (I2)
- net Y10: now also U18.13 (I12); no longer U18.11 (I11)
- net Y2: now also U18.4 (I4); no longer U18.3 (I3)
- net Y3: now also U18.5 (I5); no longer U18.4 (I4)
- net Y4: now also U18.6 (I6); no longer U18.5 (I5)
- net Y5: now also U18.7 (I7); no longer U18.6 (I6)
- net Y6: now also U18.8 (I8); no longer U18.7 (I7)
- net Y7: now also U18.9 (I9); no longer U18.8 (I8)
- net Y8: now also U18.10 (I10); no longer U18.9 (I9)
- net Y9: now also U18.11 (I11); no longer U18.10 (I10)
- net VBLANK: no longer names the net of U18.18 (IO6)
- new net !IRQ: J1.7 (Pin_7)
- new net !NMI: J1.10 (Pin_10)
- new net !P_SELECT: J1.16 (Pin_16)
- new net !READ: J1.9 (Pin_9)
- new net !RESET: J1.14 (Pin_14)
- new net !WRITE: J1.12 (Pin_12)
- new net D6: J1.39 (Pin_39)
- new net D7: J1.40 (Pin_40)
- new net PHI1: J1.5 (Pin_5)
- new net PHI2: J1.8 (Pin_8)
- new net RDY: J1.13 (Pin_13)
- no-connect marks 20 -> 38
Other:
- moved on the sheet: J3

Commit message: Revert "Integtrate IO into mail board, begion VGA layout"
This reverts commit 15baf3f71fbe492a9e0b6e5b5ec863db56e31855.
Parts:
- removed J1, J2: Conn_02x20_Odd_Even, Connector_PinSocket_2.54mm:PinSocket_2x20_P2.54mm_Vertical, symbol Connector_Generic:Conn_02x20_Odd_Even
- J?: renamed from J3; footprint Connector_Dsub:DSUB-15-HD_Female_Horizontal_P2.29x1.98mm_EdgePinOffset3.03mm_Housed_MountingHolesOffset4.94mm -> (none)
- R1, R2, R3, R4, R5, R6: footprint Resistor_THT:R_Axial_DIN0207_L6.3mm_D2.5mm_P10.16mm_Horizontal -> (none)
Connections:
- net !HRST: now also U17.17 (IO7); no longer U17.21 (I03)
- net !VRST: now also U18.17 (IO7); no longer U18.20 (IO4)
- net BLANK: now also U18.16 (IO8); no longer U18.21 (I03)
- net CLK: now also U17.3 (I3); no longer U17.4 (I4)
- net HBLANK: now also U17.18 (IO6), U18.13 (I12); no longer U17.22 (IO2), U18.23 (IO1)
- net HSYNC: now also U17.19 (IO5); no longer U17.23 (IO1)
- net LINE_INC: now also U17.16 (IO8); no longer U17.20 (IO4)
- net VCLK: no longer U17.1 (I1/CLK), U18.1 (I1/CLK)
- net VSYNC: now also U18.19 (IO5); no longer U18.22 (IO2)
- net X0: now also U17.1 (I1/CLK); no longer U17.2 (I2)
- net X1: now also U17.2 (I2); no longer U17.3 (I3)
- net X10: now also U17.11 (I11); no longer U17.13 (I12)
- net X3: now also U17.4 (I4); no longer U17.5 (I5)
- net X4: now also U17.5 (I5); no longer U17.6 (I6)
- net X5: now also U17.6 (I6); no longer U17.7 (I7)
- net X6: now also U17.7 (I7); no longer U17.8 (I8)
- net X7: now also U17.8 (I8); no longer U17.9 (I9)
- net X8: now also U17.9 (I9); no longer U17.10 (I10)
- net X9: now also U17.10 (I10); no longer U17.11 (I11)
- net Y0: now also U18.1 (I1/CLK); no longer U18.2 (I2)
- net Y1: now also U18.2 (I2); no longer U18.3 (I3)
- net Y10: now also U18.11 (I11); no longer U18.13 (I12)
- net Y2: now also U18.3 (I3); no longer U18.4 (I4)
- net Y3: now also U18.4 (I4); no longer U18.5 (I5)
- net Y4: now also U18.5 (I5); no longer U18.6 (I6)
- net Y5: now also U18.6 (I6); no longer U18.7 (I7)
- net Y6: now also U18.7 (I7); no longer U18.8 (I8)
- net Y7: now also U18.8 (I8); no longer U18.9 (I9)
- net Y8: now also U18.9 (I9); no longer U18.10 (I10)
- net Y9: now also U18.10 (I10); no longer U18.11 (I11)
- net VBLANK: now reaches U18.18 (IO6)
- new net HBLANK_END: U17.20 (IO4)
- new net HBLANK_START: U17.21 (I03)
- new net HSYNC_END: U17.22 (IO2)
- new net HSYNC_START: U17.23 (IO1)
- new net VBLANK_END: U18.20 (IO4)
- new net VBLANK_START: U18.21 (I03)
- new net VSYNC_END: U18.22 (IO2)
- new net VSYNC_START: U18.23 (IO1)
- no-connect marks 38 -> 20
Other:
- moved on the sheet: J?
