File: vga-board/vga-board.sch (KiCad schematic (older format))
At the start: 30 parts, among them U10 74HC163, U11 74LS158, U17 GAL22V10, U18 GAL22V10, U4 74HC373, U5 74HC373, U6 74HC373, U7 74HC373, U8 71256SA12TPG, X1 40MHz

Commit message: More on VGA
Parts:
- U12: renamed from U?; footprint (none) -> Package_DIP:DIP-16_W7.62mm_Socket
- gave numbers to parts that had none: 16
Connections:
- net labels added: CLK, HBLANK_END, HBLANK_START, HSYNC_END, HSYNC_START, VBLANK, VBLANK_END, VBLANK_START, VSYNC_END, VSYNC_START
- wire segments 52 -> 53
- no-connect marks 15 -> 16
Other:
- note added: "40MHz square wave video clock"
- note added: "The GAL takes the X coordinate and generates HSYNC, HBLANK.\nAdditionally, it resets the X counter and incrementsthe Y counter after X=1055"
- note added: "The GAL takes the Y coordinate and generates VSYNC and VBLANK.\nAdditionally it resets the Y counter after Y=627.\nAdditionally it combines HBLANK and VBLANK to generate BLANK."
- note added: "The video RAM. This accepts addresses from a\nvariery of sources. It usually outputs data but\nnot during the CPU master stage. !VRAM_WRITE\nonly strobes low when the CPU has exclusive\naccess to the RAM and is attempting a write."
- note added: "This video card outputs SVGA at 800x600 using a 40MHz pixel clock. It displays a 100 x 37 array of 8x16 characters,\neach with 4-bit RGBI foreground and background colours. Characters are RAM based and therefore are fully\ncustomizable and must be supplied by the CPU at boot. It masters the CPU clock drives the CPU at 5MHz.\n\nThe circuit is in theory capable of displaying 1024 x 768 (128x48) but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"
- note added: "Truth Table - VRAM_WRITE is additionally dependent on R!W(LOW) and A15(HIGH)"
- note added: "X2 drives the CPU at 5MHz"
- note removed: "The video RAM. This accepts addresses from a variery of sources.\nIt usually outputs data but not during the CPU master stage.\n!VRAM_WRITE only strobes low when the CPU has exclusive\naccess to the RAM and is attempting a write."
- note removed: "This GAL takes the X coordinate and generates HSYNC, HBLANK.\nAdditionally, it resets the X counter and incrementsthe Y counter after X=1055"
- note removed: "This GAL takes the Y coordinate and generates VSYNC and VBLANK.\nAdditionally it resets the Y counter after Y=627.\nAdditionally it combines HBLANK and VBLANK to generate BLANK."
- moved on the sheet: R1, R2, R3, R4, R5, R6

Commit message: Add VGA socket, fix routing errors on CPU board
Parts:
- added J?: DB15_Female_HighDensity, symbol Connector:DB15_Female_HighDensity
Connections:
- wire segments 53 -> 69
- no-connect marks 16 -> 20
Changed lines of the file:
@@
 Text Notes 850  10650 0    50   ~ 0
 This video card outputs SVGA at 800x600 using a 40MHz pixel clock. It displays a 100 x 37 array of 8x16 characters,\neach with 4-bit RGBI foreground and background colours. Characters are RAM based and therefore are fully\ncustomizable and must be supplied by the CPU at boot. It masters the CPU clock drives the CPU at 5MHz.\n\nThe circuit is in theory capable of displaying 1024 x 768 (128x48) but I couldn't find a through-hole 65MHz\noscillator. I am also worried about running the CPU at 8+MHZ without an upgraded ROM.
+$Comp
+L Connector:DB15_Female_HighDensity J?
+U 1 1 5FE4F9CB
+P 15050 7200
+F 0 "J?" H 15050 8067 50  0000 C CNN
+F 1 "DB15_Female_HighDensity" H 15050 7976 50  0000 C CNN
+F 2 "" H 14100 7600 50  0001 C CNN
+F 3 " ~" H 14100 7600 50  0001 C CNN
+	1    15050 7200
+	1    0    0    -1
+$EndComp
+$Comp
+L power:GND #PWR?
+U 1 1 5FE5F12B
+P 14500 7600
+F 0 "#PWR?" H 14500 7350 50  0001 C CNN
+F 1 "GND" H 14500 7450 50  0000 C CNN
+F 2 "" H 14500 7600 50  0001 C CNN
+F 3 "" H 14500 7600 50  0001 C CNN
+	1    14500 7600
+	1    0    0    -1
+$EndComp
+Text GLabel 14650 6800 0    50   Input ~ 0
+R
+Text GLabel 14650 7000 0    50   Input ~ 0
+G
+Text GLabel 14650 7200 0    50   Input ~ 0
+B
+Text GLabel 15450 7200 2    50   Input ~ 0
+HSYNC
+Text GLabel 15450 7400 2    50   Input ~ 0
+VSYNC
+Wire Wire Line
+	15450 7400 15350 7400
+Wire Wire Line
+	15350 7200 15450 7200
+Wire Wire Line
+	14650 7200 14750 7200
+Wire Wire Line
+	14650 7000 14750 7000
+Wire Wire Line
+	14650 6800 14750 6800
+Wire Wire Line
+	14750 7600 14500 7600
+Wire Wire Line
+	14500 6700 14750 6700
+Wire Wire Line
+	14500 6900 14750 6900
+Connection ~ 14500 6900
+Wire Wire Line
+	14500 6900 14500 6700
+Wire Wire Line
+	14500 7100 14750 7100
+Connection ~ 14500 7100
+Wire Wire Line
+	14500 7100 14500 6900
+Wire Wire Line
+	14500 7300 14750 7300
+Connection ~ 14500 7300
+Wire Wire Line
+	14500 7300 14500 7100
+Wire Wire Line
+	14500 7600 14500 7500
+Wire Wire Line
+	14500 7500 14750 7500
+Connection ~ 14500 7500
+Wire Wire Line
+	14500 7500 14500 7300
+NoConn ~ 14750 7400
+NoConn ~ 15350 6800
+NoConn ~ 15350 7000
+NoConn ~ 15350 7600
+Connection ~ 14500 7600
 $EndSCHEMATC

Commit message: Design new VGA board
Parts:
- removed U1, U13, U14, U15, U3, U9: 74HC244, Package_DIP:DIP-20_W7.62mm_Socket, symbol 74xx:74HC244
- added C1, C10, C11, C12, C13, C14, C15, C16, C17, C18, C19, C2, C20, C21, C22, C23, C24, C25, C3, C4, C5, C6, C7, C8, C9: 0.1uF, Capacitor_THT:C_Disc_D6.0mm_W2.5mm_P5.00mm, symbol Device:C
- added J1, J2: EXP, Connector_PinHeader_2.54mm:PinHeader_2x20_P2.54mm_Vertical, symbol Connector_Generic:Conn_02x20_Odd_Even
- added U11, U12, U14, U15, U16, U17, U24, U25: 74HC373, Package_DIP:DIP-20_W7.62mm_Socket, symbol 74xx:74HC373
- J3: renamed from J?; value DB15_Female_HighDensity -> VGA; footprint (none) -> Connector_Dsub:DSUB-15-HD_Female_Horizontal_P2.29x1.98mm_EdgePinOffset3.03mm_Housed_MountingHolesOffset4.94mm
- R1, R6: footprint (none) -> Resistor_THT:R_Axial_DIN0207_L6.3mm_D2.5mm_P10.16mm_Horizontal
- R2: renamed from R4; footprint (none) -> Resistor_THT:R_Axial_DIN0207_L6.3mm_D2.5mm_P10.16mm_Horizontal
- R3: renamed from R2; footprint (none) -> Resistor_THT:R_Axial_DIN0207_L6.3mm_D2.5mm_P10.16mm_Horizontal
- R4: renamed from R5; footprint (none) -> Resistor_THT:R_Axial_DIN0207_L6.3mm_D2.5mm_P10.16mm_Horizontal
- R5: renamed from R3; footprint (none) -> Resistor_THT:R_Axial_DIN0207_L6.3mm_D2.5mm_P10.16mm_Horizontal
- renumbered U17 to U1, U23 to U10, U4 to U13, U6 to U18, U2 to U19, U10 to U2, U12 to U20, U5 to U21, U7 to U22, U11 to U23, U20 to U3, U22 to U4, U8 to U5, U16 to U6, U18 to U7, U19 to U8, U21 to U9
Connections:
- net labels added: !IRQ, !NMI, !P_SELECT, !READ, !RESET, !WRITE, BLANK_OUT, D6, D7, HSYNC_OUT, PHI1, PHI2, RDY, VSYNC_OUT
- net labels removed: HBLANK, HBLANK_END, HBLANK_START, HSYNC_END, HSYNC_START, VBLANK_END, VBLANK_START, VSYNC_END, VSYNC_START
- wire segments 69 -> 130
- no-connect marks 20 -> 59
Other:
- note added: "Character / colour address buffer (active when !CC_MASTER is low).\nThese buffers address the video RAM when fetching the character code or colour.\nThe first 8kB of RAM (VA14=0, VA13=0) contains the character selection.\nThe next 8kB (VA14=0, VA13=1) contains the colour selection.\nThe location is determined by the most significant bits of the pixel coordinates."
- note added: "The GAL takes the X coordinate and generates HSYNC, HBLANK.\nAdditionally, it resets the X counter and incrementsthe Y counter after X=1055\nAdditionally it combines HBLANK and VBLANK to generate BLANK."
- note added: "The GAL takes the Y coordinate and generates VSYNC and VBLANK.\nAdditionally it resets the Y counter after Y=627."
- note added: "The character latch has a dual purpose. During the character fetch, it latches a character code.\nDuring the font fetch, it addresses the video RAM to fetch the appropriate character font.\nThis selects font RAM (VA14=1, VA13=0) and buffers the appropriate line (based on the least\nsignificant part of the Y coordinate.) of the appropriate character (selected by the character latch)."
- note added: "The colour latch operates in 2 stages. First, during the colour fetch stage, the colours\nare stored in the first latch. Then when RELATCH goes high, the colour is moved into\nthe active latch at the same time as the character data."
- note added: "The font latch operates in 2 stages. First, during the font fetch, 8 pixels (one row) of\nthe font is loaded into the first latch. Then when RELATCH does high, the row is\nloaded into the second active latch. From there is is serialized by the multiplexer."
- note added: "This GAL is the main timing logic and primarily controls video RAM access\n\nThe video (pixel) clock runs at 40MHz and is divided to ultimately produce a CPU clock of 5MHz. During each 5MHz (200ns) cycle, 8 pixels are\ndisplayed and 4 memory accesses occur - 50ns each.\n\n1) Character fetch. During this stage, the XY coordinates are used to address video RAM and latch the next character to displa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"
- note added: "This circuit selects either the foreground or background colour depending\non the active pixel, or black is BLANK_OUT is asserted. The selected 4-bit\ncolour is then converted to an analog voltage (0v, 0.45v or 0.7v)."
- note added: "This pair of latches caches HSYNC and VSYNC ready to be output. As with the other outputs, this\nis a 2-stage process ensuring that all outputs change simultaneosly with RELATCH is asserted."
- note added: "This video card outputs SVGA at 800x600 using a 40MHz pixel clock. It displays a 100 x 37 array of 8x16 characters,\neach with 4-bit RGBI foreground and background colours. Characters are RAM based and therefore are fully\ncustomizable and must be supplied by the CPU at boot. It masters the CPU clock drives the CPU at 5MHz."
- note removed: "Character / colour address buffer (active when !CC_MASTER is low).\nThese buffers address the video RAM when fetching the character code or colour.\nThe first 8kB of RAM (A14=0, A13=0) contains the character selection.\nThe next 8kB (A14=0, A13=1) contains the colour selection.\nThe location is determined by the most significant bits of the pixel coordinates."
- note removed: "Font address buffer"
- note removed: "The GAL takes the X coordinate and generates HSYNC, HBLANK.\nAdditionally, it resets the X counter and incrementsthe Y counter after X=1055"
- note removed: "The GAL takes the Y coordinate and generates VSYNC and VBLANK.\nAdditionally it resets the Y counter after Y=627.\nAdditionally it combines HBLANK and VBLANK to generate BLANK."
- note removed: "The character latch has a dual purpose. During the character fetch, it latches a character code.\nDuring the font fetch, it addresses the video RAM to fetch the appropriate character font.\nThe second half of the font address buffer selects the font RAM (A14=1, A13=0)\nand buffers the appropriate line of the character based on the least significant part of the Y coordinate."
- note removed: "The colour latch operates in 2 stages. First, during the colour fetch stage, the colours\nare stored in the first latch. Then when RELATCH goes high, the colour is moved into\nthe active latch at the same time the character is loaded into the serializer."
- note removed: "The font latch operated in 2 stages. First, during the font fetch, 8 pixels (one row) of\nthe font is loaded into the first latch. Then when RELATCH does high, the row is\nloaded into the second active latch. From there is is serialized by the multiplexer."
- note removed: "This GAL is the main timing logic and primarily controls video RAM access\n\nThe video (pixel) clock runs at 40MHz and is divided to ultimately produce a CPU clock of 5MHz. During each 5MHz (200ns) cycle, 8 pixels are\ndisplayed and 4 memory accesses occur - 50ns each.\n\n1) Character access. During this stage, the XY coordinates are used to address video RAM and latch the next character to displ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"
- note removed: "This circuit selects either the foreground or background colour depending on\nthe active pixel, or black is BLANK is set (LOW). The selected 4-bit colour is\nthen converted to an analog voltage (0v, 0.45v or 0.7v)."
- note removed: "This video card outputs SVGA at 800x600 using a 40MHz pixel clock. It displays a 100 x 37 array of 8x16 characters,\neach with 4-bit RGBI foreground and background colours. Characters are RAM based and therefore are fully\ncustomizable and must be supplied by the CPU at boot. It masters the CPU clock drives the CPU at 5MHz.\n\nThe circuit is in theory capable of displaying 1024 x 768 (128x48) but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"
- moved on the sheet: J3, R1, R2, R3, R4, R5, R6

Commit message: remove old peripheral boards, begn new vga design
Parts:
- removed C19, C20, C21, C22, C23, C24, C25: 0.1uF, Capacitor_THT:C_Disc_D6.0mm_W2.5mm_P5.00mm, symbol Device:C
- removed J3: VGA, Connector_Dsub:DSUB-15-HD_Female_Horizontal_P2.29x1.98mm_EdgePinOffset3.03mm_Housed_MountingHolesOffset4.94mm, symbol Connector:DB15_Female_HighDensity
- removed R1, R3, R5: 680R, Resistor_THT:R_Axial_DIN0207_L6.3mm_D2.5mm_P10.16mm_Horizontal, symbol Device:R
- removed R2, R4, R6: 1.2k, Resistor_THT:R_Axial_DIN0207_L6.3mm_D2.5mm_P10.16mm_Horizontal, symbol Device:R
- removed U1, U6, U7: GAL22V10, Package_DIP:DIP-24_W7.62mm_Socket, symbol computer:GAL22V10
- removed U10, U2, U3, U4, U8, U9: 74HC163, Package_DIP:DIP-16_W7.62mm_Socket, symbol 74xx:74LS163
- removed U11, U12, U13, U14, U15, U16, U17, U18, U19, U21, U22, U24, U25: 74HC373, Package_DIP:DIP-20_W7.62mm_Socket, symbol 74xx:74HC373
- removed U20: 74LS251, Package_DIP:DIP-16_W7.62mm_Socket, symbol 74xx:74LS251
- removed U23: 74LS158, Package_DIP:DIP-16_W7.62mm_Socket, symbol 74xx:74LS158
- removed U5: 71256SA12TPG, Package_DIP:DIP-28_W7.62mm_Socket, symbol Memory_RAM:CY62256-70PC
- removed X1: 40MHz, Oscillator:Oscillator_DIP-8, symbol Oscillator:VC-81
- added U1: XC95144XL-TQ100, Package_QFP:TQFP-100_14x14mm_P0.5mm, symbol CPLD_Xilinx:XC95144XL-TQ100
- added U2: IS61C5128AL-10TLI, Package_SO:TSOP-II-44_10.16x18.41mm_P0.8mm, symbol Memory_RAM:IS61C5128AL-10TLI
- added X1: 50MHz, Oscillator:Oscillator_DIP-8, symbol Oscillator:VC-83
- C1, C11, C13, C15, C17, C3, C5, C7, C9: value 0.1uF -> 100n; footprint Capacitor_THT:C_Disc_D6.0mm_W2.5mm_P5.00mm -> Capacitor_SMD:C_0402_1005Metric
- C10, C12, C14, C16, C18, C2, C4, C6, C8: value 0.1uF -> 10n; footprint Capacitor_THT:C_Disc_D6.0mm_W2.5mm_P5.00mm -> Capacitor_SMD:C_0402_1005Metric
Connections:
- net labels added: +3V3, CLK_V, VA15, VA16, VA17, VA18, VOE, VWE
- net labels removed: !CC_MASTER, !CPU_MASTER, !FONT_MASTER, !HRST, !P_SELECT, !VRAM_WRITE, !VRST, B, BG_B, BG_G, BG_I, BG_R, BLANK, BLANK_OUT, CHAR_LATCH, COLOR, COLOR_LATCH, CPU_MASTER, FG_B, FG_I, FG_R, FONT_LATCH, G, HSYNC, HSYNC_OUT, LINE_INC, PIXEL, R, RELATCH, VBLANK, VCLK, VSYNC, VSYNC_OUT, X0, X1, X10, X2, X3, X4, X5, X6, X7, X8, X9, Y0, Y1, Y10, Y2, Y3, Y4, Y5, Y6, Y7, Y8, Y9
- wire segments 130 -> 47
- no-connect marks 59 -> 1
Other:
- note removed: "40MHz square wave video clock"
- note removed: "CPU access buffer (active when !CPU_MASTER is low)\nFor the final 1/4 of the 5MHz CPU cycle, the CPU has exclusive access to video RAM."
- note removed: "Character / colour address buffer (active when !CC_MASTER is low).\nThese buffers address the video RAM when fetching the character code or colour.\nThe first 8kB of RAM (VA14=0, VA13=0) contains the character selection.\nThe next 8kB (VA14=0, VA13=1) contains the colour selection.\nThe location is determined by the most significant bits of the pixel coordinates."
- note removed: "Character latch"
- note removed: "Colour latch A"
- note removed: "Colour latch B"
- note removed: "Font latch A"
- note removed: "Font latch B"
- note removed: "Font serializer"
- note removed: "Pixel colour selector"
- note removed: "Simple counter for X pixel position incremented on every rising edge of VCLK."
- note removed: "Simple counter for Y pixel position incremented every time LINE_INC is set."
- note removed: "The GAL takes the X coordinate and generates HSYNC, HBLANK.\nAdditionally, it resets the X counter and incrementsthe Y counter after X=1055\nAdditionally it combines HBLANK and VBLANK to generate BLANK."
- note removed: "The GAL takes the Y coordinate and generates VSYNC and VBLANK.\nAdditionally it resets the Y counter after Y=627."
- note removed: "The character latch has a dual purpose. During the character fetch, it latches a character code.\nDuring the font fetch, it addresses the video RAM to fetch the appropriate character font.\nThis selects font RAM (VA14=1, VA13=0) and buffers the appropriate line (based on the least\nsignificant part of the Y coordinate.) of the appropriate character (selected by the character latch)."
- note removed: "The colour latch operates in 2 stages. First, during the colour fetch stage, the colours\nare stored in the first latch. Then when RELATCH goes high, the colour is moved into\nthe active latch at the same time as the character data."
- note removed: "The font latch operates in 2 stages. First, during the font fetch, 8 pixels (one row) of\nthe font is loaded into the first latch. Then when RELATCH does high, the row is\nloaded into the second active latch. From there is is serialized by the multiplexer."
- note removed: "The video RAM. This accepts addresses from a\nvariery of sources. It usually outputs data but\nnot during the CPU master stage. !VRAM_WRITE\nonly strobes low when the CPU has exclusive\naccess to the RAM and is attempting a write."
- note removed: "This GAL is the main timing logic and primarily controls video RAM access\n\nThe video (pixel) clock runs at 40MHz and is divided to ultimately produce a CPU clock of 5MHz. During each 5MHz (200ns) cycle, 8 pixels are\ndisplayed and 4 memory accesses occur - 50ns each.\n\n1) Character fetch. During this stage, the XY coordinates are used to address video RAM and latch the next character to displa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"
- note removed: "This circuit selects either the foreground or background colour depending\non the active pixel, or black is BLANK_OUT is asserted. The selected 4-bit\ncolour is then converted to an analog voltage (0v, 0.45v or 0.7v)."
- note removed: "This pair of latches caches HSYNC and VSYNC ready to be output. As with the other outputs, this\nis a 2-stage process ensuring that all outputs change simultaneosly with RELATCH is asserted."
- note removed: "This video card outputs SVGA at 800x600 using a 40MHz pixel clock. It displays a 100 x 37 array of 8x16 characters,\neach with 4-bit RGBI foreground and background colours. Characters are RAM based and therefore are fully\ncustomizable and must be supplied by the CPU at boot. It masters the CPU clock drives the CPU at 5MHz."
- note removed: "Truth Table - VRAM_WRITE is additionally dependent on R!W(LOW) and A15(HIGH)"
- note removed: "X2 drives the CPU at 5MHz"
- moved on the sheet: J1, J2

Commit message: continue new vga
Parts:
- added J3: Conn_02x05_Odd_Even, Connector_IDC:IDC-Header_2x05_P2.54mm_Vertical, symbol Connector_Generic:Conn_02x05_Odd_Even
Connections:
- net +3V3: now also J3.4 (Pin_4)
- net GND: now also J3.10 (Pin_10), J3.2 (Pin_2)
- net TDI: now reaches U1.45 (TDI)
- net TDI: now also J3.9 (Pin_9)
- net TMS: now reaches U1.47 (TMS)
- net TMS: now also J3.5 (Pin_5)
- net TCK: now reaches U1.48 (TCK)
- net TCK: now also J3.1 (Pin_1)
- net TDO: now reaches U1.83 (TDO)
- net TDO: now also J3.3 (Pin_3)
- no-connect marks 1 -> 4
Changed lines of the file:
@@
 Text GLabel 3700 3950 2    50   BiDi ~ 0
 VD5
+$Comp
+L power:+3V3 #PWR0102
+U 1 1 5FFA207D
+P 5750 5100
+F 0 "#PWR0102" H 5750 4950 50  0001 C CNN
+F 1 "+3V3" V 5765 5228 50  0000 L CNN
+F 2 "" H 5750 5100 50  0001 C CNN
+F 3 "" H 5750 5100 50  0001 C CNN
+	1    5750 5100
+	0    1    1    0
+$EndComp
+$Comp
+L power:GND #PWR0103
+U 1 1 5FFA3434
+P 5750 5400
+F 0 "#PWR0103" H 5750 5150 50  0001 C CNN
+F 1 "GND" V 5755 5272 50  0000 R CNN
+F 2 "" H 5750 5400 50  0001 C CNN
+F 3 "" H 5750 5400 50  0001 C CNN
+	1    5750 5400
+	0    -1   -1   0
+$EndComp
+$Comp
+L Connector_Generic:Conn_02x05_Odd_Even J3
+U 1 1 5FFA4B8B
+P 5450 5200
+F 0 "J3" H 5500 5617 50  0000 C CNN
+F 1 "Conn_02x05_Odd_Even" H 5500 5526 50  0000 C CNN
+F 2 "Connector_IDC:IDC-Header_2x05_P2.54mm_Vertical" H 5450 5200 50  0001 C CNN
+F 3 "~" H 5450 5200 50  0001 C CNN
+	1    5450 5200
+	1    0    0    -1
+$EndComp
+Text GLabel 3700 6350 2    50   Input ~ 0
+TCK
+Text GLabel 3700 6150 2    50   Input ~ 0
+TDI
+Text GLabel 3700 6450 2    50   Output ~ 0
+TDO
+Text GLabel 3700 6250 2    50   Input ~ 0
+TMS
+Text GLabel 5250 5000 0    50   Output ~ 0
+TCK
+Text GLabel 5250 5100 0    50   Input ~ 0
+TDO
+Text GLabel 5250 5200 0    50   Output ~ 0
+TMS
+Text GLabel 5250 5400 0    50   Output ~ 0
+TDI
+NoConn ~ 5250 5300
+NoConn ~ 5750 5300
+$Comp
+L power:GND #PWR0104
+U 1 1 5FFB4C0A
+P 5750 5000
+F 0 "#PWR0104" H 5750 4750 50  0001 C CNN
+F 1 "GND" V 5755 4872 50  0000 R CNN
+F 2 "" H 5750 5000 50  0001 C CNN
+F 3 "" H 5750 5000 50  0001 C CNN
+	1    5750 5000
+	0    -1   -1   0
+$EndComp
+NoConn ~ 5750 5200
 $EndSCHEMATC

Commit message: more vga board routing
Parts:
- removed X1: 50MHz, Oscillator:Oscillator_DIP-8, symbol Oscillator:VC-83
- added C19: 100n, Capacitor_SMD:C_0402_1005Metric, symbol Device:C
- added C20: 10n, Capacitor_SMD:C_0402_1005Metric, symbol Device:C
- added J4: DB15_Female_HighDensity, Connector_Dsub:DSUB-15-HD_Female_Horizontal_P2.29x1.98mm_EdgePinOffset3.03mm_Housed_MountingHolesOffset4.94mm, symbol Connector:DB15_Female_HighDensity
- added R1, R10, R11, R12, R14, R15, R16, R17, R18, R19, R2, R21, R3, R4, R5, R6, R8, R9: 560R, Resistor_SMD:R_0402_1005Metric, symbol Device:R
- added R13, R20, R7: 47R, Resistor_SMD:R_0402_1005Metric, symbol Device:R
- added X1: ABLNO, Oscillator:Oscillator_SMD_Abracon_ASV-4Pin_7.0x5.1mm, symbol Oscillator:ABLNO
Connections:
- net !RESET: now also U1.1 (I/O/GTS3)
- net +3V3: now also C19.1, C20.1, X1.1 (Vctrl), X1.4 (VDD)
- net A0: now also U1.3 (I/O/GTS1); no longer U1.1 (I/O/GTS3)
- net A1: now also U1.4 (I/O/GTS2); no longer U1.2 (I/O/GTS4)
- net A10: now also U1.14 (P14); no longer U1.13 (P13)
- net A11: now also U1.15 (P15); no longer U1.14 (P14)
- net A12: now also U1.16 (P16); no longer U1.15 (P15)
- net A13: now also U1.17 (P17); no longer U1.16 (P16)
- net A14: now also U1.18 (P18); no longer U1.17 (P17)
- net A15: now also U1.19 (P19); no longer U1.18 (P18)
- net A2: now also U1.6 (P6); no longer U1.3 (I/O/GTS1)
- net A3: now also U1.7 (P7); no longer U1.4 (I/O/GTS2)
- net A4: now also U1.8 (P8); no longer U1.6 (P6)
- net A5: now also U1.9 (P9); no longer U1.7 (P7)
- net A6: now also U1.10 (P10); no longer U1.8 (P8)
- net A7: now also U1.11 (P11); no longer U1.9 (P9)
- net A8: now also U1.12 (P12); no longer U1.11 (P11)
- net A9: now also U1.13 (P13); no longer U1.12 (P12)
- net CLK_V: now also U1.27 (I/O/GCK3), X1.3 (RFout); no longer U1.22 (I/O/GCK1)
- net D0: now also U1.20 (P20); no longer U1.24 (P24)
- net D1: now also U1.22 (I/O/GCK1); no longer U1.25 (P25)
- net D2: now also U1.25 (P25); no longer U1.27 (I/O/GCK3)
- net D3: now also U1.24 (P24); no longer U1.28 (P28)
- net D5: now also U1.28 (P28); no longer U1.30 (P30)
- net D7: now also U1.30 (P30); no longer U1.33 (P33)
- net GND: now also C19.2, C20.2, R12.2, R19.2, R5.2, X1.2 (GND)
- net R!W: now also U1.2 (I/O/GTS4)
- net HSYNC: now reaches U1.90 (P90)
- net HSYNC: now also J4.13
- net VSYNC: now reaches U1.91 (P91)
- net VSYNC: now also J4.14
- net B0: now reaches U1.92 (P92)
- net B0: now also R16.2
- net B1: now reaches U1.93 (P93)
- net B1: now also R15.2
- net G0: now reaches U1.94 (P94)
- net G0: now also R9.2
- net G1: now reaches U1.95 (P95)
- net G1: now also R8.2
- net R0: now reaches U1.96 (P96)
- net R0: now also R2.2
- net R1: now reaches U1.97 (P97)
- net R1: now also R1.2
- new net: R1.1, R3.2, R4.1, R6.2
- new net: R2.1, R4.2, R5.1
- new net: R3.1, R6.1, R7.2
- new net: R10.2, R11.1, R14.2, R8.1
- new net: R11.2, R12.1, R9.1
- new net: R10.1, R13.2, R14.1
- new net: R15.1, R17.2, R18.1, R21.2
- new net: R16.1, R18.2, R19.1
- new net: R17.1, R20.2, R21.1
- new net: J4.10, J4.5, J4.6, J4.7, J4.8, J4.9
- new net B: J4.3, R20.1
- new net G: J4.2, R13.1
- new net R: J4.1, R7.1
- no-connect marks 4 -> 3
Other:
- moved on the sheet: C1, C10, C11, C12, C13, C14, C15, C16, C2, C3, C4, C5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
